Commit message: Add materials to install

File: bluerov2_description/urdf/apriltag_panel.xacro (robot description, xacro)
@@ -14,5 +14,7 @@
           <box size="0.15 0.15 0.001"/>
         </geometry>
-        <material name="white">
+        <material name="apriltag">
+          <!-- Replace the following with the correct path to your PNG file -->
+          <texture filename="package://bluerov2_description/materials/textures/tag36_11_00038.png"/>
           <color rgba="1 1 1 1"/>
         </material>

Commit message: Added tag to robot!

File: bluerov2_description/urdf/apriltag_panel.xacro (robot description, xacro)
@@ -12,9 +12,9 @@
         <origin xyz="0 0 0" rpy="0 0 0"/>
         <geometry>
-          <box size="0.15 0.15 0.001"/>
+          <mesh filename="package://bluerov2_description/meshes/apriltag_panel.dae"/>
         </geometry>
         <material name="apriltag">
           <!-- Replace the following with the correct path to your PNG file -->
-          <texture filename="package://bluerov2_description/materials/textures/tag36_11_00038.png"/>
+          <texture filename="package://bluerov2_description/materials/textures/tag36_11_00037.png"/>
           <color rgba="1 1 1 1"/>
         </material>
@@ -32,4 +32,21 @@
       <origin xyz="0 ${y_offset} 0" rpy="${PI/2} 0 0"/>
     </joint>
+    <!-- Add Gazebo-specific material configuration -->
+    <gazebo reference="${ns}/apriltag_panel">
+      <visual>
+        <material>
+          <ambient>1 1 1 1</ambient>
+          <diffuse>1 1 1 1</diffuse>
+          <specular>0.1 0.1 0.1 1</specular>
+          <pbr>
+            <metal>
+              <albedo_map>package://bluerov2_description/materials/textures/tag36_11_00037.png</albedo_map>
+              <roughness>0.8</roughness>
+              <metalness>0.1</metalness>
+            </metal>
+          </pbr>
+        </material>
+      </visual>
+    </gazebo>
   </xacro:macro>
 </xacro>

Commit message: Decrease freq, increase res of camera image. Add additional tags

File: bluerov2_description/urdf/apriltag_panel.xacro (robot description, xacro)
@@ -2,6 +2,6 @@
 <xacro xmlns:xacro="http://www.ros.org/wiki/xacro">
   <xacro:property name="PI" value="3.1415927"/>
-  <xacro:macro name="apriltag_panel" params="ns y_offset">
-    <link name="${ns}/apriltag_panel">
+  <xacro:macro name="apriltag_panel" params="ns panel_name:=side *origin">
+    <link name="${ns}/apriltag_panel_${panel_name}">
       <inertial>
         <mass value="0.01"/>
@@ -27,11 +27,11 @@
       </collision>
     </link>
-    <joint name="${ns}/apriltag_panel_joint" type="fixed">
+    <joint name="${ns}/apriltag_panel_${panel_name}_joint" type="fixed">
       <parent link="${ns}/base_link"/>
-      <child link="${ns}/apriltag_panel"/>
-      <origin xyz="0 ${y_offset} 0" rpy="${PI/2} 0 0"/>
+      <child link="${ns}/apriltag_panel_${panel_name}"/>
+      <xacro:insert_block name="origin"/>
     </joint>
     <!-- Add Gazebo-specific material configuration -->
-    <gazebo reference="${ns}/apriltag_panel">
+    <gazebo reference="${ns}/apriltag_panel_${panel_name}">
       <visual>
         <material>

File: bluerov2_description/urdf/bluerov2.xacro (robot description, xacro)
@@ -61,6 +61,17 @@
 <xacro:include filename="sensors.xacro"/>
 <xacro:include filename="apriltag_panel.xacro"/>
-<!-- Add the AprilTag panel -->
-<xacro:apriltag_panel ns="${ns}" y_offset="${y_size/2 + 0.045}"/>
+<!-- Add the AprilTag panels -->
+<xacro:apriltag_panel ns="${ns}" panel_name="left">
+  <origin xyz="0 ${y_size/2 + 0.045} 0" rpy="${PI/2} 0 0"/>
+</xacro:apriltag_panel>
+<xacro:apriltag_panel ns="${ns}" panel_name="right">
+  <origin xyz="0 ${-y_size/2 - 0.045} 0" rpy="${PI/2} 0 0"/>
+</xacro:apriltag_panel>
+<xacro:apriltag_panel ns="${ns}" panel_name="back">
+  <origin xyz="${-x_size/2 - 0.045} 0 0" rpy="${PI/2} 0 ${PI/2}"/>
+</xacro:apriltag_panel>
+<xacro:apriltag_panel ns="${ns}" panel_name="front">
+  <origin xyz="${x_size/2 + 0.045} 0 0" rpy="${PI/2} 0 ${-PI/2}"/>
+</xacro:apriltag_panel>
 <!-- other Gazebo plugins -->
 <xacro:if value="$(arg simulation)">

File: bluerov2_description/urdf/sensors.xacro (robot description, xacro)
@@ -195,6 +195,6 @@
     <horizontal_fov>1.047</horizontal_fov>
     <image>
-        <width>640</width>
-        <height>400</height>
+        <width>1280</width>
+        <height>720</height>
     </image>
     <clip>
@@ -204,5 +204,5 @@
     </camera>
     <always_on>1</always_on>
-    <update_rate>30</update_rate>
+    <update_rate>10</update_rate>
     <visualize>true</visualize>
     <topic>${ns}/image</topic>

Commit message: Added all april tags

File: bluerov2_description/urdf/apriltag_panel.xacro (robot description, xacro)
@@ -12,8 +12,7 @@
         <origin xyz="0 0 0" rpy="0 0 0"/>
         <geometry>
-          <mesh filename="package://bluerov2_description/meshes/apriltag_panel.dae"/>
+          <box size="0.15 0.15 0.001"/>
         </geometry>
         <material name="apriltag">
-          <!-- Replace the following with the correct path to your PNG file -->
           <texture filename="package://bluerov2_description/materials/textures/tag36_11_00037.png"/>
           <color rgba="1 1 1 1"/>

File: bluerov2_description/urdf/bluerov2.xacro (robot description, xacro)
@@ -63,20 +63,20 @@
 <!-- Add the AprilTag panels -->
 <xacro:apriltag_panel ns="${ns}" panel_name="left">
-  <origin xyz="0 ${y_size/2 + 0.045} 0" rpy="${PI/2} 0 0"/>
+  <origin xyz="0 ${y_size/2 + 0.045} 0" rpy="${PI/2} ${PI/2} 0"/>
 </xacro:apriltag_panel>
 <xacro:apriltag_panel ns="${ns}" panel_name="right">
-  <origin xyz="0 ${-y_size/2 - 0.045} 0" rpy="${PI/2} 0 0"/>
+  <origin xyz="0 ${-y_size/2 - 0.045} 0" rpy="${PI/2} ${PI/2} ${PI}"/>
 </xacro:apriltag_panel>
 <xacro:apriltag_panel ns="${ns}" panel_name="back">
-  <origin xyz="${-x_size/2 - 0.045} 0 0" rpy="${PI/2} 0 ${PI/2}"/>
+  <origin xyz="${-x_size/2 - 0.045} 0 0" rpy="${PI/2} ${PI/2} ${PI/2}"/>
 </xacro:apriltag_panel>
 <xacro:apriltag_panel ns="${ns}" panel_name="front">
-  <origin xyz="${x_size/2 + 0.045} 0 0" rpy="${PI/2} 0 ${-PI/2}"/>
+  <origin xyz="${x_size/2 + 0.045} 0 0" rpy="${PI/2} ${PI/2} ${-PI/2}"/>
 </xacro:apriltag_panel>
 <xacro:apriltag_panel ns="${ns}" panel_name="top">
-  <origin xyz="0 0 ${z_size/2 + 0.045}" rpy="0 0 0"/>
+  <origin xyz="0 0 ${z_size/2 + 0.045}" rpy="0 0 ${PI}"/>
 </xacro:apriltag_panel>
 <xacro:apriltag_panel ns="${ns}" panel_name="bottom">
-  <origin xyz="0 0 ${-z_size/2 - 0.045}" rpy="${PI} 0 0"/>
+  <origin xyz="0 0 ${-z_size/2 - 0.045 - 0.10}" rpy="${PI} 0 0"/>
 </xacro:apriltag_panel>
 <!-- other Gazebo plugins -->
